File: gatchaspFlex.kicad_pcb (KiCad board)
At the start: 2 copper layers, 46.2 x 76 mm, 22 parts

Commit message: Add files via upload
Parts:
- moved SPK3 19.5 mm to (201.8, 149.2)
- moved SPK4 13.3 mm to (213.1, 149.1)
Routing:
- net Net-(SPK1-Pad1): track 89.7 -> 121.6 mm
- net Net-(SPK2-Pad1): track 95.4 -> 111.4 mm
- net Net-(TP13-Pad1): track 91.5 -> 92.0 mm
Other:
- board size 46.2 x 76 mm -> 46.6 x 90.3 mm

Commit message: Add files via upload
Parts:
- TP4, TP5, TP6, TP7: footprint SparkFun-Connector:TestPoint-0.75mm -> Connector_Wire:SolderWirePad_1x01_SMD_1x2mm
- moved TP4 0.70 mm to (182.7, 65.0)
- moved TP5 0.70 mm to (179.5, 65.0)
- moved TP6 0.70 mm to (181.1, 65.0)
- moved TP7 0.60 mm to (184.6, 62.8), turned to -90 degrees
- moved GND1 0.50 mm to (215.2, 62.5)
Routing:
- net Net-(TP15-Pad1): track 90.2 -> 92.0 mm
- net Net-(TP12-Pad1): track 96.4 -> 97.2 mm

Commit message: Add files via upload
Parts:
- moved SPK3 3.00 mm to (201.8, 146.2)
- moved SPK4 3.00 mm to (213.1, 146.1)
- moved GND1 2.58 mm to (217.8, 62.5)
- moved TP2 2.12 mm to (192.1, 103.5)
- moved TP3 2.12 mm to (193.9, 103.5)
- moved TP0 1.58 mm to (210.6, 66.8)
- moved SPK1 1.12 mm to (179.5, 82.5)
- moved SPK2 1.12 mm to (182.6, 82.5)
- moved TP1 0.50 mm to (198.8, 68.7)
Routing:
- net Net-(SPK1-Pad1): track 121.6 -> 116.8 mm
- net Net-(SPK2-Pad1): track 111.4 -> 107.6 mm
- net Net-(GND1-Pad1): track 125.9 -> 128.2 mm
- net Net-(TP11-Pad1): track 73.2 -> 75.3 mm
- net Net-(TP10-Pad1): track 72.5 -> 74.6 mm
- net Net-(TP0-Pad1): track 108.2 -> 109.4 mm
Other:
- board size 46.6 x 90.3 mm -> 48.2 x 88.3 mm
